Commit message: renamed launch files and updated screen pose detection

File: dicemaster_central/resource/dice.urdf (robot description, URDF)
Before this commit: robot dice_master, 37 links, 36 joints
Links:
- added link imu_link, mass 0.01; collision box size=0.02 0.02 0.005; visual box size=0.02 0.02 0.005
Joints:
- added joint imu_joint: type fixed, parent base_link, child imu_link, origin xyz=0 0 0 rpy=0 0 0

Commit message: made working dice urdf

File: dicemaster_central/resource/dice.urdf (robot description, URDF)
Before this commit: robot dice_master, 38 links, 37 joints
Joints:
- joint screen_2_joint: origin xyz=0 0.0508 0 rpy=1.5708 0 0 -> xyz=0 0.0508 0 rpy=1.5708 0 3.14159
- joint screen_3_joint: origin xyz=0.0508 0 0 rpy=0 1.5708 0 -> xyz=0.0508 0 0 rpy=1.5708 0 1.5708
- joint screen_5_joint: origin xyz=-0.0508 0 0 rpy=0 -1.5708 0 -> xyz=-0.0508 0 0 rpy=1.5708 0 -1.5708
- joint screen_6_joint: origin xyz=0 0 -0.0508 rpy=3.14159 0 0 -> xyz=0 0 -0.0508 rpy=0 0 3.14159

Commit message: made working screen orientation detection

File: dicemaster_central/resource/dice.urdf (robot description, URDF)
Before this commit: robot dice_master, 38 links, 37 joints
Joints:
- joint screen_1_edge_left_joint: origin xyz=0 -0.0475 0.001 rpy=0 0 0 -> xyz=0 0.0475 0.001 rpy=0 0 0
- joint screen_1_edge_right_joint: origin xyz=0 0.0475 0.001 rpy=0 0 0 -> xyz=0 -0.0475 0.001 rpy=0 0 0
- joint screen_2_edge_left_joint: origin xyz=0 -0.0475 0.001 rpy=0 0 0 -> xyz=0 0.0475 0.001 rpy=0 0 0
- joint screen_2_edge_right_joint: origin xyz=0 0.0475 0.001 rpy=0 0 0 -> xyz=0 -0.0475 0.001 rpy=0 0 0
- joint screen_2_joint: origin xyz=0 0.0508 0 rpy=1.5708 0 3.14159 -> xyz=0.0508 0 0 rpy=1.5708 0 1.5708
- joint screen_3_edge_left_joint: origin xyz=0 -0.0475 0.001 rpy=0 0 0 -> xyz=0 0.0475 0.001 rpy=0 0 0
- joint screen_3_edge_right_joint: origin xyz=0 0.0475 0.001 rpy=0 0 0 -> xyz=0 -0.0475 0.001 rpy=0 0 0
- joint screen_3_joint: origin xyz=0.0508 0 0 rpy=1.5708 0 1.5708 -> xyz=0 0.0508 0 rpy=1.5708 0 3.14159
- joint screen_4_edge_left_joint: origin xyz=0 -0.0475 0.001 rpy=0 0 0 -> xyz=0 0.0475 0.001 rpy=0 0 0
- joint screen_4_edge_right_joint: origin xyz=0 0.0475 0.001 rpy=0 0 0 -> xyz=0 -0.0475 0.001 rpy=0 0 0
- joint screen_4_joint: origin xyz=0 -0.0508 0 rpy=-1.5708 0 0 -> xyz=-0.0508 0 0 rpy=1.5708 0 -1.5708
- joint screen_5_edge_left_joint: origin xyz=0 -0.0475 0.001 rpy=0 0 0 -> xyz=0 0.0475 0.001 rpy=0 0 0
- joint screen_5_edge_right_joint: origin xyz=0 0.0475 0.001 rpy=0 0 0 -> xyz=0 -0.0475 0.001 rpy=0 0 0
- joint screen_5_joint: origin xyz=-0.0508 0 0 rpy=1.5708 0 -1.5708 -> xyz=0 -0.0508 0 rpy=1.5708 0 0
- joint screen_6_edge_left_joint: origin xyz=0 -0.0475 0.001 rpy=0 0 0 -> xyz=0 0.0475 0.001 rpy=0 0 0
- joint screen_6_edge_right_joint: origin xyz=0 0.0475 0.001 rpy=0 0 0 -> xyz=0 -0.0475 0.001 rpy=0 0 0
- joint screen_6_joint: origin xyz=0 0 -0.0508 rpy=0 0 3.14159 -> xyz=0 0 -0.0508 rpy=3.14159 0 3.14159

File: dicemaster_central/resource/dice.urdf.xacro (robot description, xacro)
@@ -55,31 +55,31 @@
     <origin xyz="0 0 0.0508" rpy="0 0 0"/> <!-- Half cube height up -->
   </joint>
-  <!-- Screen 2: Right face (+Y direction) -->
-  <xacro:screen_component screen_id="2" color_r="0.0" color_g="0.0" color_b="1.0"/> <!-- Blue -->
+  <!-- Screen 3: Back face (+X direction) -->
+  <xacro:screen_component screen_id="2" color_r="0.0" color_g="1.0" color_b="0.0"/> <!-- Green -->
   <joint name="screen_2_joint" type="fixed">
     <parent link="base_link"/>
     <child link="screen_2_link"/>
-    <origin xyz="0 0.0508 0" rpy="1.5708 0 3.14159"/> <!-- Rotated to face +Y -->
+    <origin xyz="0.0508 0 0" rpy="1.5708 0 1.5708"/> <!-- Rotated to face +X -->
   </joint>
-  <!-- Screen 3: Back face (+X direction) -->
-  <xacro:screen_component screen_id="3" color_r="0.0" color_g="1.0" color_b="0.0"/> <!-- Green -->
+  <!-- Screen 2: Right face (+Y direction) -->
+  <xacro:screen_component screen_id="3" color_r="0.0" color_g="0.0" color_b="1.0"/> <!-- Blue -->
   <joint name="screen_3_joint" type="fixed">
     <parent link="base_link"/>
     <child link="screen_3_link"/>
-    <origin xyz="0.0508 0 0" rpy="1.5708 0 1.5708"/> <!-- Rotated to face +X -->
+    <origin xyz="0 0.0508 0" rpy="1.5708 0 3.14159"/> <!-- Rotated to face +Y -->
   </joint>
-  <!-- Screen 4: Left face (-Y direction) -->
-  <xacro:screen_component screen_id="4" color_r="1.0" color_g="0.0" color_b="1.0"/> <!-- Magenta -->
+  <!-- Screen 5: Front face (-X direction) -->
+  <xacro:screen_component screen_id="4" color_r="1.0" color_g="1.0" color_b="0.0"/> <!-- Yellow -->
   <joint name="screen_4_joint" type="fixed">
     <parent link="base_link"/>
     <child link="screen_4_link"/>
-    <origin xyz="0 -0.0508 0" rpy="-1.5708 0 0"/> <!-- Rotated to face -Y -->
+    <origin xyz="-0.0508 0 0" rpy="1.5708 0 -1.5708"/> <!-- Rotated to face -X -->
   </joint>
-  <!-- Screen 5: Front face (-X direction) -->
-  <xacro:screen_component screen_id="5" color_r="1.0" color_g="1.0" color_b="0.0"/> <!-- Yellow -->
+  <!-- Screen 4: Left face (-Y direction) -->
+  <xacro:screen_component screen_id="5" color_r="1.0" color_g="0.0" color_b="1.0"/> <!-- Magenta -->
   <joint name="screen_5_joint" type="fixed">
     <parent link="base_link"/>
     <child link="screen_5_link"/>
-    <origin xyz="-0.0508 0 0" rpy="1.5708 0 -1.5708"/> <!-- Rotated to face -X -->
+    <origin xyz="0 -0.0508 0" rpy="1.5708 0 0"/> <!-- Rotated to face -Y -->
   </joint>
   <!-- Screen 6: Bottom face (-Z direction) -->
@@ -88,5 +88,5 @@
     <parent link="base_link"/>
     <child link="screen_6_link"/>
-    <origin xyz="0 0 -0.0508" rpy="0 0 3.14159"/> <!-- Half cube height down, flipped -->
+    <origin xyz="0 0 -0.0508" rpy="3.14159 0 3.14159"/> <!-- Half cube height down, flipped -->
   </joint>
 </robot>

File: dicemaster_central/resource/screen_component.urdf.xacro (robot description, xacro)
@@ -35,10 +35,10 @@
     <link name="screen_${screen_id}_edge_top"/>
     <!-- Right edge (+Y direction in screen local frame) -->
-    <joint name="screen_${screen_id}_edge_right_joint" type="fixed">
+    <joint name="screen_${screen_id}_edge_left_joint" type="fixed">
       <parent link="screen_${screen_id}_link"/>
-      <child link="screen_${screen_id}_edge_right"/>
+      <child link="screen_${screen_id}_edge_left"/>
       <origin xyz="0 0.0475 0.001" rpy="0 0 0"/>
     </joint>
-    <link name="screen_${screen_id}_edge_right"/>
+    <link name="screen_${screen_id}_edge_left"/>
     <!-- Bottom edge (-X direction in screen local frame) -->
     <joint name="screen_${screen_id}_edge_bottom_joint" type="fixed">
@@ -49,10 +49,10 @@
     <link name="screen_${screen_id}_edge_bottom"/>
     <!-- Left edge (-Y direction in screen local frame) -->
-    <joint name="screen_${screen_id}_edge_left_joint" type="fixed">
+    <joint name="screen_${screen_id}_edge_right_joint" type="fixed">
       <parent link="screen_${screen_id}_link"/>
-      <child link="screen_${screen_id}_edge_left"/>
+      <child link="screen_${screen_id}_edge_right"/>
       <origin xyz="0 -0.0475 0.001" rpy="0 0 0"/>
     </joint>
-    <link name="screen_${screen_id}_edge_left"/>
+    <link name="screen_${screen_id}_edge_right"/>
   </xacro:macro>
 </robot>

Commit message: Updated URDF for demo version assembly

File: dicemaster_central/resource/dice.urdf (robot description, URDF)
Before this commit: robot dice_master, 38 links, 37 joints
Joints:
- removed joint imu_joint
- added joint base_joint: type fixed, parent imu_link, child base_link, origin xyz=0 0 0 rpy=-3.14159 0 3.14159
- joint screen_2_joint: origin xyz=0.0508 0 0 rpy=1.5708 0 1.5708 -> xyz=0 0.0508 0 rpy=-1.5708 0 0
- joint screen_3_joint: origin xyz=0 0.0508 0 rpy=1.5708 0 3.14159 -> xyz=-0.0508 0 0 rpy=0 -1.5708 0
- joint screen_4_joint: origin xyz=-0.0508 0 0 rpy=1.5708 0 -1.5708 -> xyz=0 -0.0508 0 rpy=0 1.5708 -1.5708
- joint screen_5_joint: origin xyz=0 -0.0508 0 rpy=1.5708 0 0 -> xyz=0.0508 0 0 rpy=0 -1.5708 3.14159

File: dicemaster_central/resource/dice.urdf.xacro (robot description, xacro)
@@ -3,5 +3,30 @@
   <!-- Include the screen component macro -->
   <xacro:include filename="screen_component.urdf.xacro"/>
-  <!-- Base link (center of the dice) -->
+  <!-- IMU link (root link of the robot) -->
+  <link name="imu_link">
+    <visual>
+      <geometry>
+        <box size="0.02 0.02 0.005"/> <!-- Small IMU sensor -->
+      </geometry>
+      <material name="imu_sensor">
+        <color rgba="0.3 0.3 0.3 0.9"/> <!-- Dark gray for IMU -->
+      </material>
+    </visual>
+    <collision>
+      <geometry>
+        <box size="0.02 0.02 0.005"/>
+      </geometry>
+    </collision>
+    <inertial>
+      <mass value="0.01"/>
+      <inertia ixx="0.0001" ixy="0" ixz="0" iyy="0.0001" iyz="0" izz="0.0001"/>
+    </inertial>
+  </link>
+  <!-- Base link (center of the dice, attached to IMU) -->
+  <joint name="base_joint" type="fixed">
+    <parent link="imu_link"/>
+    <child link="base_link"/>
+    <origin xyz="0 0 0" rpy="-3.14159 0 3.14159"/> <!-- Base at center of IMU, no rotation -->
+  </joint>
   <link name="base_link">
     <visual>
@@ -23,29 +48,4 @@
     </inertial>
   </link>
-  <!-- IMU link (at center of dice, aligned with base_link) -->
-  <joint name="imu_joint" type="fixed">
-    <parent link="base_link"/>
-    <child link="imu_link"/>
-    <origin xyz="0 0 0" rpy="0 0 0"/> <!-- IMU at center of dice -->
-  </joint>
-  <link name="imu_link">
-    <visual>
-      <geometry>
-        <box size="0.02 0.02 0.005"/> <!-- Small IMU sensor -->
-      </geometry>
-      <material name="imu_sensor">
-        <color rgba="0.3 0.3 0.3 0.9"/> <!-- Dark gray for IMU -->
-      </material>
-    </visual>
-    <collision>
-      <geometry>
-        <box size="0.02 0.02 0.005"/>
-      </geometry>
-    </collision>
-    <inertial>
-      <mass value="0.01"/>
-      <inertia ixx="0.0001" ixy="0" ixz="0" iyy="0.0001" iyz="0" izz="0.0001"/>
-    </inertial>
-  </link>
   <!-- Screen 1: Top face (+Z direction) -->
   <xacro:screen_component screen_id="1" color_r="1.0" color_g="0.0" color_b="0.0"/> <!-- Red -->
@@ -55,31 +55,31 @@
     <origin xyz="0 0 0.0508" rpy="0 0 0"/> <!-- Half cube height up -->
   </joint>
-  <!-- Screen 3: Back face (+X direction) -->
+  <!-- Screen 2: Right face (+Y direction) -->
   <xacro:screen_component screen_id="2" color_r="0.0" color_g="1.0" color_b="0.0"/> <!-- Green -->
   <joint name="screen_2_joint" type="fixed">
     <parent link="base_link"/>
     <child link="screen_2_link"/>
-    <origin xyz="0.0508 0 0" rpy="1.5708 0 1.5708"/> <!-- Rotated to face +X -->
+    <origin xyz="0 0.0508 0" rpy="-1.5708 0 0"/> <!-- Rotated to face +Y -->
   </joint>
-  <!-- Screen 2: Right face (+Y direction) -->
+  <!-- Screen 3: Front face (-X direction) -->
   <xacro:screen_component screen_id="3" color_r="0.0" color_g="0.0" color_b="1.0"/> <!-- Blue -->
   <joint name="screen_3_joint" type="fixed">
     <parent link="base_link"/>
     <child link="screen_3_link"/>
-    <origin xyz="0 0.0508 0" rpy="1.5708 0 3.14159"/> <!-- Rotated to face +Y -->
+    <origin xyz="-0.0508 0 0" rpy="0 -1.5708 0"/> <!-- Rotated to face -X -->
   </joint>
-  <!-- Screen 5: Front face (-X direction) -->
+  <!-- Screen 4: Left face (-Y direction) -->
   <xacro:screen_component screen_id="4" color_r="1.0" color_g="1.0" color_b="0.0"/> <!-- Yellow -->
   <joint name="screen_4_joint" type="fixed">
     <parent link="base_link"/>
     <child link="screen_4_link"/>
-    <origin xyz="-0.0508 0 0" rpy="1.5708 0 -1.5708"/> <!-- Rotated to face -X -->
+    <origin xyz="0 -0.0508 0" rpy="0 1.5708 -1.5708"/> <!-- Rotated to face -Y -->
   </joint>
-  <!-- Screen 4: Left face (-Y direction) -->
+  <!-- Screen 5: Back face (+X direction) -->
   <xacro:screen_component screen_id="5" color_r="1.0" color_g="0.0" color_b="1.0"/> <!-- Magenta -->
   <joint name="screen_5_joint" type="fixed">
     <parent link="base_link"/>
     <child link="screen_5_link"/>
-    <origin xyz="0 -0.0508 0" rpy="1.5708 0 0"/> <!-- Rotated to face -Y -->
+    <origin xyz="0.0508 0 0" rpy="0 -1.5708 3.14159"/> <!-- Rotated to face +X -->
   </joint>
   <!-- Screen 6: Bottom face (-Z direction) -->
